File: Media-Macroboard/Media-Macroboard.kicad_sch (KiCad schematic)
At the start: 25 parts, among them IC1 MCP73871-4CCI_ML, IC2 LM1117MPX-33NOPB, J1 SS-52400-002, J2 B2B-PH-SM4-TB_LF__SN_

Commit message: First productable version
Parts:
- C4, C6: footprint Capacitor_SMD:C_0805_2012Metric_Pad1.18x1.45mm_HandSolder -> Capacitor_SMD:C_1206_3216Metric
Changed lines of the file:
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@@
 			)
 		)
-		(property "Footprint" "Capacitor_SMD:C_0805_2012Metric_Pad1.18x1.45mm_HandSolder"
+		(property "Footprint" "Capacitor_SMD:C_1206_3216Metric"
 			(at 45.4152 137.16 0)
 			(effects
@@
 			)
 		)
-		(property "Footprint" "Capacitor_SMD:C_0805_2012Metric_Pad1.18x1.45mm_HandSolder"
+		(property "Footprint" "Capacitor_SMD:C_1206_3216Metric"
 			(at 92.4052 137.16 0)
 			(effects
